Commit message: error fix

File: final_project/urdf/turtlebot3_burger.gazebo.xacro (robot description, xacro)
@@ -126,5 +126,5 @@
 					rpy="0 0 0"/>
 			<geometry>
-                <mesh filename="package://turtlebot3_description/meshes/sensors/webcam.dae" scale="1.0 1.0 1.0"/>
+                <mesh filename="package://final_project/meshes/sensors/webcam.dae" scale="1.0 1.0 1.0"/>
 			</geometry>
 		</visual>

File: final_project/urdf/turtlebot3_burger.urdf.xacro (robot description, xacro)
@@ -13,5 +13,5 @@
       <origin xyz="-0.032 0 0.0" rpy="0 0 0"/>
       <geometry>
-        <mesh filename="package://turtlebot3_description/meshes/bases/burger_base.stl" scale="0.001 0.001 0.001"/>
+        <mesh filename="package://final_project/meshes/bases/burger_base.stl" scale="0.001 0.001 0.001"/>
       </geometry>
       <material name="light_black"/>
